File: Torch/torch-lts.kicad_sch (KiCad schematic)
At the start: 5 parts, among them SW1 SW_SPDT

Commit message: update for BSidesKC
Parts:
- removed SW1: SW_SPDT, BadgePirates:SW_Slide_1P2T_CK_TH, symbol Switch:SW_SPDT
- added SW1: SW_Push_Dual_x2, BadgePirates:SW_PUSH_6mm_H5mm, symbol Switch:SW_Push_Dual_x2
- BT1: footprint BadgePirates:BatteryHolder_MPD_BC2003_1x2032_Fixed -> BadgePirates:2032 Through Hold Holder
Connections:
- net at R1.1: now also SW1.2 (D)
- net at BT1.1 (+): now also SW1.1 (C)
- no-connect marks 1 -> 0

Commit message: updated Logos and Adjusted size of res, alighted footprints properly to board
Parts:
- R1: footprint Resistor_THT:R_Axial_DIN0204_L3.6mm_D1.6mm_P5.08mm_Horizontal -> Resistor_THT:R_Axial_DIN0207_L6.3mm_D2.5mm_P10.16mm_Horizontal
Changed lines of the file:
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@@
       (effects (font (size 1.27 1.27)))
     )
-    (property "Footprint" "Resistor_THT:R_Axial_DIN0204_L3.6mm_D1.6mm_P5.08mm_Horizontal" (at 151.384 85.344 90)
+    (property "Footprint" "Resistor_THT:R_Axial_DIN0207_L6.3mm_D2.5mm_P10.16mm_Horizontal" (at 151.384 85.344 90)
       (effects (font (size 1.27 1.27)) hide)
     )
